File: Eagle/poiduino7(7).sch (EAGLE design)
At the start: 20 parts, among them K1 TS-1109, Y1 16MHZ

Commit message: fix pads board
Parts:
- C1, C2: value 18pf -> 10nf
- C3, C4, C6: value 0.1uf -> 10nf
- C5: value 1uf -> 100uf
- JP1: value (none) -> jp1
- JP2: value (none) -> jp2
- JP3: value (none) -> jp3
- JP4: value (none) -> jp4
- JP5: value (none) -> jp5
- U1: value (none) -> Atmega328p
Connections:
- removed net CTS: JP1.5
- removed net N$34: JP2.1
- removed net N$38: JP2.5
Other:
- moved on the sheet: C5, JP1, K1, Y1
